File: Herfurth-MinicontH1370W_BatUpgrade/Herfurth-MinicontH1370W_BatUpgrade.kicad_sch (KiCad schematic)
At the start: 12 parts, among them J1 TYPE-C-31-M-12, U1 BQ24232, U2 AP7340-33FS4-7

Commit message: LDO
Parts:
- removed U2: AP7340-33FS4-7, Package_DFN_QFN:OnSemi_XDFN4-1EP_1.0x1.0mm_EP0.52x0.52mm, symbol minicont:AP7340-xxxx
- added C3, C5: 10u, symbol Device:C_Small
- added C4, C6: 22u, symbol Device:C_Polarized
- added R4, R6: R_Small, symbol Device:R_Small
- added R5: 4k3, Resistor_SMD:R_0603_1608Metric_Pad0.98x0.95mm_HandSolder, symbol Device:R_Small
- added TH1: 10k, Resistor_SMD:R_0603_1608Metric_Pad0.98x0.95mm_HandSolder, symbol Device:Thermistor_NTC
- added U3: AMS1117-2.5, Package_TO_SOT_SMD:SOT-223-3_TabPin2, symbol Regulator_Linear:AMS1117-2.5
- BT1: value Li 18650 -> Li
Connections:
- net +5V: no longer R3.1, U1.6 (EN1)
- net GND: now also C3.2, C4.2, C5.2, C6.2, R5.1, R6.2, TH1.1; no longer U1.15 (TD)
- net VCC: now also R3.1, U1.6 (EN1), C5.1, U3.3 (VI)
- net at U1.1 (TS): now also TH1.2
- net at U1.16 (ISET): now also R5.2
- net Charging renamed ~{Charging}
- net PGOOD renamed ~{PGOOD}
- new net: C3.1, R4.2, R6.1, U3.1 (GND)
- new net +2V5: C4.1, C6.1, R4.1, U3.2 (VO)
- no-connect marks 8 -> 11
Other:
- note added: "Battery Management"
- note added: "LDO"
- note added: "Status Indicators"
- note added: "USB-C"
- note added: "~{Charging} high if I_{Charge} < I_{Term} and until V_{In} toggled. ~{Charging} flashing at 2Hz if safety timers expired."
- note added: "~{PGOOD} low if V_{Bat}+V_{In(DT)} < V_{In} < V_{OVP}"
- moved on the sheet: BT1, C1, C2, D1, D2, D3, J1, R1, R2, R3, U1
